File: SynthControlPCB.sch (KiCad schematic (older format))
At the start: 25 parts

Commit message: continued initial design work.
Parts:
- removed C?: 0.1uF, symbol C
- removed L?: FB(30R), symbol Ferrite_Bead_Small
- removed R? (x3): 47k, symbol R
- removed SW?: RE1, symbol Rotary_Encoder_Switch
- removed U?: SAMD20G18A-AU, TQFP48, symbol SAMD20G18A-AU
- added L?: FB(30R), symbol Ferrite_Bead_Small
- added R? (x10): 47k, symbol R
- added SW? (x5): Rotary_Encoder, symbol Rotary_Encoder
- added SW?: SW_Rotary12, symbol SW_Rotary12
- added U?: SAMD20E15A-AU, TQFP32, symbol SAMD20E15A-AU
Connections:
- net +3V3: now also L?.1, R?.1, R?.1, R?.1, R?.1, R?.1, R?.1, R?.1, R?.1, R?.1, R?.1, U?.30 (VDDIN)
- net AIN2: now also U?.7 (TC1WO0/SERCOM0P2/Y4/AIN2/AIN6/PA06)
- net AIN3: now also U?.8 (TC1WO1/SERCOM0P3/Y5/AIN3/AIN7/PA07)
- net GND: now also SW?.2 (C), SW?.2 (C), SW?.2 (C), SW?.2 (C), SW?.2 (C), U?.10 (GND), U?.28 (GND)
- net PA19: now also R?.2, SW?.3 (B), U?.20 (ACCMP1/TC3WO1/SERCOM3P3/SERCOM1P3/X7/PA19)
- net PA30: now also U?.31 (GCLKIO0/SWCLK/TC1WO0/SERCOM1P2/PA30)
- net PA31: now also U?.32 (SWDIO/TC1WO1/SERCOM1P3/PA31)
- net SCK: now also U?.24 (TC5WO1/SERCOM5P3/SERCOM3P3/PA25)
- net SDA: now also U?.23 (TC5WO0/SERCOM5P2/SERCOM3P2/PA24)
- net USB_D+: now also U?.27 (GCLKIO0/PA28)
- net USB_D-: now also U?.25 (GCLKIO0/PA27)
- net ~RST: now also U?.26 (~RESET~)
- net at C?.1: now also U?.29 (VDDCORE)
- net at C?.1, C?.1: now also L?.2, U?.9 (VDDANA)
- new net AIN1: U?.6 (TC0W01/SERCOM0P1/Y3/AIN1/AIN5/PA05)
- new net AIN4: U?.5 (TC0WO0/SERCOM0P0/Y2/AIN0/AIN4/VREFB/PA04)
- new net PA08: R?.2, SW?.1 (A), U?.11 (TC0WO0/SERCOM2P0/SERCOM0P0/X0/AIN16/NMI/PA08)
- new net PA09: R?.2, SW?.3 (B), U?.12 (TC0WO1/SERCOM2P1/SERCOM0P1/X1/AIN17/PA09)
- new net PA10: R?.2, SW?.1 (A), U?.13 (GCLKIO4/TC1WO0/SERCOM2P2/SERCOM0P2/X2/AIN18/PA10)
- new net PA11: R?.2, SW?.3 (B), U?.14 (GCLKIO5/TC1WO1/SERCOM2P3/SERCOM0P3/X3/AIN19/PA11)
- new net PA14: R?.2, SW?.1 (A), U?.15 (XIN/GCLKIO0/TC3WO0/SERCOM4P2/SERCOM2P2/PA14)
- new net PA15: R?.2, SW?.3 (B), U?.16 (XOUT/GCLKIO1/TC3WO1/SERCOM4P3/SERCOM2P3/PA15)
- new net PA16: R?.2, SW?.1 (A), U?.17 (GCLKIO2/TC2WO0/SERCOM3P0/SERCOM1P0/X4/PA16)
- new net PA17: R?.2, SW?.3 (B), U?.18 (GCLKIO3/TC2WO1/SERCOM3P1/SERCOM1P1/X5/PA17)
- new net PA18: R?.2, SW?.1 (A), U?.19 (ACCMP0/TC3WO0/SERCOM3P2/SERCOM1P2/X6/PA18)
- new net PA22: U?.21 (GCLKIO6/TC4WO0/SERCOM5P0/SERCOM3P0/X10/PA22)
- new net PA23: U?.22 (GCLKIO7/TC4WO1/SERCOM5P1/SERCOM3P1/X11/PA23)
Other:
- moved on the sheet: C?, R?, U?

Commit message: continued initial design.
Parts:
- removed SW?: SW_Rotary12, symbol SW_Rotary12
- added C?: 33pF, symbol C
- added R?: 3k9, symbol R
- added R? (x2): 47k, symbol R
- added RV? (x4): POT, symbol POT
- added SW? (x3): SW_Rotary1x4, symbol SW_Rotary1x4
- added SW? (x3): SW_SP3T, symbol SW_SP3T
- added SW? (x3): SW_SPDT, symbol SW_SPDT
Connections:
- net +3V3: now also R?.1, R?.1, R?.1, RV?.1, RV?.1, RV?.1, RV?.1
- net AIN1: now also RV?.2
- net AIN2: now also RV?.2
- net AIN3: now also RV?.2
- net AIN4: now also RV?.2
- net GND: now also U?.17 (A1), U?.18 (A2), C?.2, RV?.3, RV?.3, RV?.3, RV?.3
- net SCK: now also U?.14 (SCL)
- net SDA: now also U?.15 (SDA)
- net at U?.11 (GPB5): now also SW?.4
- net at U?.12 (GPB6): now also SW?.1 (A)
- net at U?.13 (GPB7): now also SW?.3 (C)
- net at U?.16 (A0): now also R?.2
- net at U?.2 (GPB0): now also SW?.1 (x2)
- net at U?.21 (GPA0): now also SW?.1 (x2)
- net at U?.22 (GPA1): now also SW?.2 (x2)
- net at U?.23 (GPA2): now also SW?.4
- net at U?.25 (GPA4): now also SW?.1 (A)
- net at U?.26 (GPA5): now also SW?.3 (C)
- net at U?.27 (GPA6): now also SW?.1 (A)
- net at U?.28 (GPA7): now also SW?.3 (C)
- net at U?.3 (GPB1): now also SW?.2 (x2)
- net at U?.4 (GPB2): now also SW?.4
- net at U?.5 (GPB3): now also SW?.1
- net at U?.7 (GPB4): now also SW?.2
- net at U?.9 (CLK): now also C?.1, R?.2
- net at U?.11 (GPB5): now also SW?.2
- net at U?.12 (GPB6): now also SW?.3
- net at U?.13 (GPB7): now also SW?.4
- net at U?.23 (GPA2): now also SW?.3
- net at U?.24 (GPA3): now also SW?.4
- net at U?.4 (GPB2): now also SW?.3
- net at U?.5 (GPB3): now also SW?.4
- net at U?.7 (GPB4): now also SW?.1
- new net: R?.2, SW?.2 (B), SW?.2 (B), SW?.2 (B), SW?.3, SW?.3, SW?.3, SW?.5 (C), SW?.5 (C), SW?.5 (C)
Other:
- moved on the sheet: C?, R?, SW?, U?

Commit message: schematic level design just about done.  Time to start on footprints and the BOM .
Parts:
- added C1, C2: 15pF, symbol C
- added D1: D_Shockley, symbol D_Shockley
- added D2: LED, symbol LED
- added J3: USB_OTG, symbol USB_OTG
- added R2: 2k, symbol R
- added Y1: Crystal, symbol Crystal
- gave numbers to parts that had none: 52
Connections:
- net +3V3: now also R2.1
- net +5V: now also D1.1 (K)
- net GND: now also C1.1, C2.1, D2.1 (K), J3.5 (GND), J3.6 (Shield)
- net USB_D+: now also J3.3 (D+); no longer U2.27 (GCLKIO0/PA28)
- net USB_D-: now also J3.2 (D-); no longer U2.25 (GCLKIO0/PA27)
- net at U2.1 (XIN32/TC2WO0/SERCOM1P0/PA00): now also C1.2, Y1.1
- net at U2.2 (XOUT32/TC2WO1/SERCOM1P1/PA01): now also C2.2, Y1.2
- net USB_ID: now reaches U2.3 (VOUT/Y0/AIN0/PA02)
- net USB_ID: now also J3.4 (ID)
- net VRef: now reaches U2.4 (Y1/AIN1/VREFA/VREFP/PA03)
- new net: D1.2 (A), J3.1 (VBUS)
- new net: D2.2 (A), R2.2
Other:
- note added: "External crystal is optional\nAnd may not be needed \nfor this project."
- moved on the sheet: C11, R11, R16, SW10, SW12, SW13, SW14, SW7, SW8, U4

Commit message: began spec-ing parts.
Parts:
- C3: footprint (none) -> Capacitors_ThroughHole:CP_Radial_D5.0mm_P2.00mm; Critical (none) -> N; Description (none) -> CAP ALUM 47UF 20% 16V RADIAL; Source (none) -> 732-8791-1-ND; VPN (none) -> 860020372004
- J2: footprint (none) -> Pin_Headers:Pin_Header_Angled_1x02_Pitch2.54mm; Critical (none) -> N; Description (none) -> CONN HEADER R/A 2POS 2.54MM; Source (none) -> A19450-ND; VPN (none) -> 640455-2
- L1: footprint (none) -> Resistors_SMD:R_0805_HandSoldering; Critical (none) -> N; Description (none) -> FERRITE BEAD 30 OHM 0805 1LN; Source (none) -> 1276-6370-1-ND; VPN (none) -> CIS21P300NE
Changed lines of the file:
@@
 F 0 "J2" H 2100 1425 50  0000 C CNN
 F 1 "Power Input" H 2100 1125 50  0000 C CNN
-F 2 "" H 2100 1325 50  0001 C CNN
+F 2 "Pin_Headers:Pin_Header_Angled_1x02_Pitch2.54mm" H 2100 1325 50  0001 C CNN
 F 3 "" H 2100 1325 50  0001 C CNN
+F 4 "~" H 2100 1325 60  0000 C CNN "Characteristics"
+F 5 "CONN HEADER R/A 2POS 2.54MM" H 2100 1325 60  0001 C CNN "Description"
+F 6 "~" H 2100 1325 60  0001 C CNN "VName"
+F 7 "640455-2" H 2100 1325 60  0001 C CNN "VPN"
+F 8 "~" H 2100 1325 60  0001 C CNN "PackaageID"
+F 9 "A19450-ND" H 2100 1325 60  0001 C CNN "Source"
+F 10 "N" H 2100 1325 60  0001 C CNN "Critical"
+F 11 "~" H 2100 1325 60  0001 C CNN "Notes"
 	1    2100 1325
 	-1   0    0    1
@@
 F 0 "L1" H 2875 1275 50  0000 L CNN
 F 1 "FB(30R)" V 2650 1125 50  0000 L CNN
-F 2 "" V 2730 1225 50  0001 C CNN
+F 2 "Resistors_SMD:R_0805_HandSoldering" V 2730 1225 50  0001 C CNN
 F 3 "" H 2800 1225 50  0001 C CNN
+F 4 "~" H 2800 1225 60  0000 C CNN "Characteristics"
+F 5 "FERRITE BEAD 30 OHM 0805 1LN" H 2800 1225 60  0001 C CNN "Description"
+F 6 "~" H 2800 1225 60  0001 C CNN "VName"
+F 7 "CIS21P300NE" H 2800 1225 60  0001 C CNN "VPN"
+F 8 "~" H 2800 1225 60  0001 C CNN "PackaageID"
+F 9 "1276-6370-1-ND" H 2800 1225 60  0001 C CNN "Source"
+F 10 "N" H 2800 1225 60  0001 C CNN "Critical"
+F 11 "~" H 2800 1225 60  0001 C CNN "Notes"
 	1    2800 1225
 	0    1    1    0
@@
 F 0 "C3" H 3250 1550 50  0000 L CNN
 F 1 "47uF" H 3250 1350 50  0000 L CNN
-F 2 "" H 3263 1300 50  0001 C CNN
+F 2 "Capacitors_ThroughHole:CP_Radial_D5.0mm_P2.00mm" H 3263 1300 50  0001 C CNN
 F 3 "" H 3225 1450 50  0001 C CNN
+F 4 "~" H 3225 1450 60  0000 C CNN "Characteristics"
+F 5 "CAP ALUM 47UF 20% 16V RADIAL" H 3225 1450 60  0001 C CNN "Description"
+F 6 "~" H 3225 1450 60  0001 C CNN "VName"
+F 7 "860020372004" H 3225 1450 60  0001 C CNN "VPN"
+F 8 "~" H 3225 1450 60  0001 C CNN "PackaageID"
+F 9 "732-8791-1-ND" H 3225 1450 60  0001 C CNN "Source"
+F 10 "N" H 3225 1450 60  0001 C CNN "Critical"
+F 11 "~" H 3225 1450 60  0001 C CNN "Notes"
 	1    3225 1450
 	1    0    0    -1
